Commit message: feat(urdf): complete humanaopen.urdf skeleton with full kinematic tree + meshes
- 24 links / 23 joints: base (differential wheels), lift (prismatic),
  torso, head pan/tilt, left+right arms (7-DOF + gripper each)
- joint names mirror lerobot_robot_humanaopen/humanaopen.py exactly
- 26 STL meshes copied into urdf/meshes/ (HumanaOpen_stl + Open-arms-mini J1-J8)
- every link has visual mesh (mm->m scale 0.001), collision box, estimated inertial
- arm joint mapping from open-arms-mini README (J1=pan, J2=lift, J3=roll,
  J4=elbow, J5=forearm, J6=wrist flex, J7=wrist yaw, J8=gripper L/R)
- origins/inertia are estimates; mesh filenames authoritative

File: hardware/urdf/humanaopen.urdf (robot description, URDF)
Before this commit: robot humanaopen, 6 links, 5 joints
Links:
- added link left_arm_elbow_flex_link, mass 0.2; collision box size=0.14 0.05 0.05; visual mesh filename=meshes/J4 v3.stl scale=0.001 0.001 0.001
- added link left_arm_forearm_rotation_link, mass 0.2; collision box size=0.06 0.06 0.06; visual mesh filename=meshes/J5 v4.stl scale=0.001 0.001 0.001
- added link left_arm_gripper_link, mass 0.15; collision box size=0.04 0.05 0.04; visual mesh filename=meshes/1.GripperFin-V3.stl scale=0.001 0.001 0.001
- added link left_arm_shoulder_lift_link, mass 0.2; collision box size=0.14 0.05 0.05; visual mesh filename=meshes/J2 v2.stl scale=0.001 0.001 0.001
- added link left_arm_shoulder_pan_link, mass 0.2; collision box size=0.06 0.06 0.06; visual mesh filename=meshes/J1 v5.stl scale=0.001 0.001 0.001
- added link left_arm_shoulder_roll_link, mass 0.2; collision box size=0.06 0.06 0.06; visual mesh filename=meshes/J3 v2.stl scale=0.001 0.001 0.001
- added link left_arm_wrist_flex_link, mass 0.2; collision box size=0.06 0.05 0.05; visual mesh filename=meshes/J6 v6.stl scale=0.001 0.001 0.001
- added link left_arm_wrist_yaw_link, mass 0.2; collision box size=0.05 0.05 0.05; visual mesh filename=meshes/J7 v4.stl scale=0.001 0.001 0.001
- added link lift_base, mass 0.6; collision box size=0.16 0.16 0.18; visual mesh filename=meshes/14.LiftBase-V16.stl scale=0.001 0.001 0.001
- added link right_arm_elbow_flex_link, mass 0.2; collision box size=0.14 0.05 0.05; visual mesh filename=meshes/J4 v3.stl scale=0.001 0.001 0.001
- added link right_arm_forearm_rotation_link, mass 0.2; collision box size=0.06 0.06 0.06; visual mesh filename=meshes/J5 v4.stl scale=0.001 0.001 0.001
- added link right_arm_gripper_link, mass 0.15; collision box size=0.04 0.05 0.04; visual mesh filename=meshes/1.GripperFin-V3.stl scale=0.001 0.001 0.001
- added link right_arm_shoulder_lift_link, mass 0.2; collision box size=0.14 0.05 0.05; visual mesh filename=meshes/J2 v2.stl scale=0.001 0.001 0.001
- added link right_arm_shoulder_pan_link, mass 0.2; collision box size=0.06 0.06 0.06; visual mesh filename=meshes/J1 v5.stl scale=0.001 0.001 0.001
- added link right_arm_shoulder_roll_link, mass 0.2; collision box size=0.06 0.06 0.06; visual mesh filename=meshes/J3 v2.stl scale=0.001 0.001 0.001
- added link right_arm_wrist_flex_link, mass 0.2; collision box size=0.06 0.05 0.05; visual mesh filename=meshes/J6 v6.stl scale=0.001 0.001 0.001
- added link right_arm_wrist_yaw_link, mass 0.2; collision box size=0.05 0.05 0.05; visual mesh filename=meshes/J7 v4.stl scale=0.001 0.001 0.001
- added link torso, mass 1.5; collision box size=0.22 0.16 0.36; visual mesh filename=meshes/10.Torso-V23.stl scale=0.001 0.001 0.001
- link base_left_wheel: mass None -> 0.15; geometry collision cylinder length=0.02 radius=0.032; visual mesh filename=meshes/4.WheelHub.stl scale=0.001 0.001 0.001
- link base_link: mass None -> 2.0; geometry collision box size=0.20 0.20 0.10; visual mesh filename=meshes/16.ChassisServoHolder-V7.stl scale=0.001 0.001 0.001
- link base_right_wheel: mass None -> 0.15; geometry collision cylinder length=0.02 radius=0.032; visual mesh filename=meshes/4.WheelHub.stl scale=0.001 0.001 0.001
- link head_pan_link: mass None -> 0.1; geometry collision box size=0.06 0.06 0.06; visual mesh filename=meshes/12.NeckYaw_V3.stl scale=0.001 0.001 0.001
- link head_tilt_link: mass None -> 0.25; geometry collision box size=0.08 0.07 0.07; visual mesh filename=meshes/11.HeadHousing_V13.stl scale=0.001 0.001 0.001
- link lift_carriage: mass None -> 0.5; geometry collision box size=0.12 0.12 0.25; visual mesh filename=meshes/3.LiftServoMount-V22.stl scale=0.001 0.001 0.001
Joints:
- added joint left_arm_elbow_flex_joint: type revolute, parent left_arm_shoulder_roll_link, child left_arm_elbow_flex_link, origin xyz=0 0 0.05 rpy=0 0 0, axis 0 1 0, limit lower=-2.09 upper=1.57 effort=30 velocity=2.0
- added joint left_arm_forearm_rotation_joint: type revolute, parent left_arm_elbow_flex_link, child left_arm_forearm_rotation_link, origin xyz=0.1 0 0 rpy=0 0 0, axis 1 0 0, limit lower=-3.14159 upper=3.14159 effort=30 velocity=2.0
- added joint left_arm_gripper_joint: type prismatic, parent left_arm_wrist_yaw_link, child left_arm_gripper_link, origin xyz=0.03 0 0 rpy=0 0 0, axis 0 0 1, limit lower=0.0 upper=0.02 effort=20 velocity=0.5
- added joint left_arm_shoulder_lift_joint: type revolute, parent left_arm_shoulder_pan_link, child left_arm_shoulder_lift_link, origin xyz=0 0 0.035 rpy=0 0 0, axis 0 1 0, limit lower=-1.57 upper=1.57 effort=30 velocity=2.0
- added joint left_arm_shoulder_pan_joint: type revolute, parent torso, child left_arm_shoulder_pan_link, origin xyz=0.115 0 0.42 rpy=0 0 0, axis 0 0 1, limit lower=-2.967 upper=2.967 effort=30 velocity=2.0
- added joint left_arm_shoulder_roll_joint: type revolute, parent left_arm_shoulder_lift_link, child left_arm_shoulder_roll_link, origin xyz=0.09 0 0 rpy=0 0 0, axis 1 0 0, limit lower=-1.57 upper=1.57 effort=30 velocity=2.0
- added joint left_arm_wrist_flex_joint: type revolute, parent left_arm_forearm_rotation_link, child left_arm_wrist_flex_link, origin xyz=0.03 0 0 rpy=0 0 0, axis 0 1 0, limit lower=-1.57 upper=1.57 effort=30 velocity=2.0
- added joint left_arm_wrist_yaw_joint: type revolute, parent left_arm_wrist_flex_link, child left_arm_wrist_yaw_link, origin xyz=0.04 0 0 rpy=0 0 0, axis 1 0 0, limit lower=-3.14159 upper=3.14159 effort=30 velocity=2.0
- added joint lift_base_joint: type fixed, parent base_link, child lift_base, origin xyz=0 0 0.08 rpy=0 0 0
- added joint right_arm_elbow_flex_joint: type revolute, parent right_arm_shoulder_roll_link, child right_arm_elbow_flex_link, origin xyz=0 0 0.05 rpy=0 0 0, axis 0 1 0, limit lower=-2.09 upper=1.57 effort=30 velocity=2.0
- added joint right_arm_forearm_rotation_joint: type revolute, parent right_arm_elbow_flex_link, child right_arm_forearm_rotation_link, origin xyz=0.1 0 0 rpy=0 0 0, axis 1 0 0, limit lower=-3.14159 upper=3.14159 effort=30 velocity=2.0
- added joint right_arm_gripper_joint: type prismatic, parent right_arm_wrist_yaw_link, child right_arm_gripper_link, origin xyz=0.03 0 0 rpy=0 0 0, axis 0 0 1, limit lower=0.0 upper=0.02 effort=20 velocity=0.5
- added joint right_arm_shoulder_lift_joint: type revolute, parent right_arm_shoulder_pan_link, child right_arm_shoulder_lift_link, origin xyz=0 0 0.035 rpy=0 0 0, axis 0 1 0, limit lower=-1.57 upper=1.57 effort=30 velocity=2.0
- added joint right_arm_shoulder_pan_joint: type revolute, parent torso, child right_arm_shoulder_pan_link, origin xyz=-0.115 0 0.42 rpy=0 0 0, axis 0 0 1, limit lower=-2.967 upper=2.967 effort=30 velocity=2.0
- added joint right_arm_shoulder_roll_joint: type revolute, parent right_arm_shoulder_lift_link, child right_arm_shoulder_roll_link, origin xyz=0.09 0 0 rpy=0 0 0, axis 1 0 0, limit lower=-1.57 upper=1.57 effort=30 velocity=2.0
- added joint right_arm_wrist_flex_joint: type revolute, parent right_arm_forearm_rotation_link, child right_arm_wrist_flex_link, origin xyz=0.03 0 0 rpy=0 0 0, axis 0 1 0, limit lower=-1.57 upper=1.57 effort=30 velocity=2.0
- added joint right_arm_wrist_yaw_joint: type revolute, parent right_arm_wrist_flex_link, child right_arm_wrist_yaw_link, origin xyz=0.04 0 0 rpy=0 0 0, axis 1 0 0, limit lower=-3.14159 upper=3.14159 effort=30 velocity=2.0
- added joint torso_joint: type fixed, parent lift_carriage, child torso, origin xyz=0 0 0.28 rpy=0 0 0
- joint base_left_wheel_joint: axis (none) -> 0 1 0; origin xyz=0 0 0 rpy=0 0 0 -> xyz=0.09 0 0 rpy=0 0 0
- joint base_right_wheel_joint: axis (none) -> 0 1 0; origin xyz=0 0 0 rpy=0 0 0 -> xyz=-0.09 0 0 rpy=0 0 0
- joint head_pan: axis (none) -> 0 0 1; origin xyz=0 0 0 rpy=0 0 0 -> xyz=0 0 0.52 rpy=0 0 0; parent lift_carriage -> torso
- joint head_tilt: axis (none) -> 0 1 0; origin xyz=0 0 0 rpy=0 0 0 -> xyz=0 0 0.03 rpy=0 0 0
- joint lift_axis: origin xyz=0 0 0 rpy=0 0 0 -> xyz=0 0 0.25 rpy=0 0 0; parent base_link -> lift_base

Commit message: fix(urdf): correct mesh origins & mirror right arm
- body STL meshes recentred: HumanaOpen CAD exports had geometry at
  (165,160)mm in each file's XY quadrant; visual origins now compensate
  so chassis/lift/torso/head sit centred on their link frames
- wheels lowered to ground (z=0.032) instead of embedded in chassis
- right arm joint X offsets mirrored (shoulder_roll/forearm/wrist/gripper)
  so it no longer crosses the torso midline
- gripper fins mounted on inboard side of each J8 jaw (L/R symmetric)
- verified with check_urdf + per-mesh world-center audit (arms now
  mirror-symmetric, chassis centred, wheels on ground)

File: hardware/urdf/humanaopen.urdf (robot description, URDF)
Before this commit: robot humanaopen, 24 links, 23 joints
Joints:
- joint base_left_wheel_joint: origin xyz=0.09 0 0 rpy=0 0 0 -> xyz=0.09 0.0 0.032 rpy=0 0 0
- joint base_right_wheel_joint: origin xyz=-0.09 0 0 rpy=0 0 0 -> xyz=-0.09 0.0 0.032 rpy=0 0 0
- joint right_arm_forearm_rotation_joint: origin xyz=0.1 0 0 rpy=0 0 0 -> xyz=-0.1 0.0 0.0 rpy=0 0 0
- joint right_arm_gripper_joint: origin xyz=0.03 0 0 rpy=0 0 0 -> xyz=-0.03 0.0 0.0 rpy=0 0 0
- joint right_arm_shoulder_roll_joint: origin xyz=0.09 0 0 rpy=0 0 0 -> xyz=-0.09 0.0 0.0 rpy=0 0 0
- joint right_arm_wrist_flex_joint: origin xyz=0.03 0 0 rpy=0 0 0 -> xyz=-0.03 0.0 0.0 rpy=0 0 0
- joint right_arm_wrist_yaw_joint: origin xyz=0.04 0 0 rpy=0 0 0 -> xyz=-0.04 0.0 0.0 rpy=0 0 0

Commit message: fix(urdf): physical grounding - wheels support chassis
Dynamic test (PyBullet) exposed: base_link collision box (0.20x0.20x0.10
centred at z=0) sat directly on the ground and lifted the wheels off it,
so the robot could not drive.

- base_link collision shrunk to 0.18x0.18x0.06 at z=0.03, clearing the
  wheel wells
- wheel collision cylinders oriented along roll axis (Y) via rpy
- verified in sim: chassis has zero ground contact, both wheels carry the
  load (3/2 contacts), robot drives +0.26m in 2.5s, lift + arms work,
  stays stable through motions

File: hardware/urdf/humanaopen.urdf (robot description, URDF)
Before this commit: robot humanaopen, 24 links, 23 joints
Links:
- link base_link: geometry collision box size=0.18 0.18 0.06; visual mesh filename=meshes/16.ChassisServoHolder-V7.stl scale=0.001 0.001 0.001
